File: PCB-Variant-A/EnvPico-nRF52840.kicad_pcb (KiCad board)
At the start: 2 copper layers, 21.2 x 57.7 mm, 48 parts, among them J3 2.54mm header 01x20, J4 2.54mm header 01x20, J5 Conn_01x03_Male, U1 LM3671MF 3.3, U2 BQ24072RGT, U3 nRF52840, Y1 32MHz 12pF

Commit message: made a couple of pcb variants for future use maybe
Connections:
- U2 pad 12: (no net) -> unconnected-(U2-Pad12)
- U2 pad 14: (no net) -> unconnected-(U2-Pad14)
- U2 pad 7: (no net) -> unconnected-(U2-Pad7)
- U3 pad A18: (no net) -> unconnected-(U3-PadA18)
- U3 pad AC11: (no net) -> unconnected-(U3-PadAC11)
- U3 pad AC15: (no net) -> unconnected-(U3-PadAC15)
- U3 pad AC17: (no net) -> unconnected-(U3-PadAC17)
- U3 pad AC19: (no net) -> unconnected-(U3-PadAC19)
- U3 pad AC9: (no net) -> unconnected-(U3-PadAC9)
- U3 pad B11: (no net) -> unconnected-(U3-PadB11)
- U3 pad B13: (no net) -> unconnected-(U3-PadB13)
- U3 pad B15: (no net) -> unconnected-(U3-PadB15)
- U3 pad B17: (no net) -> unconnected-(U3-PadB17)
- U3 pad B9: (no net) -> unconnected-(U3-PadB9)
- U3 pad F2: (no net) -> unconnected-(U3-PadF2)
- U3 pad H2: (no net) -> unconnected-(U3-PadH2)
- U3 pad J24: (no net) -> unconnected-(U3-PadJ24)
- U3 pad K2: (no net) -> unconnected-(U3-PadK2)
- U3 pad M2: (no net) -> unconnected-(U3-PadM2)
- U3 pad P2: (no net) -> unconnected-(U3-PadP2)
- U3 pad P23: (no net) -> unconnected-(U3-PadP23)
- U3 pad T23: (no net) -> unconnected-(U3-PadT23)
- U3 pad V23: (no net) -> unconnected-(U3-PadV23)
- U3 pad Y23: (no net) -> unconnected-(U3-PadY23)
- USB1 pad 3: (no net) -> unconnected-(USB1-Pad3)
- USB1 pad 9: (no net) -> unconnected-(USB1-Pad9)

Commit message: started re-design of board.
Parts:
- removed C13: 0402 1pF, Capacitor_SMD:C_0402_1005Metric
- removed C8: 0402 1.5pF, Capacitor_SMD:C_0402_1005Metric
- removed NT1: Net-Tie_2, NetTie:NetTie-2_SMD_Pad0.5mm
- removed R1: 0R 0402, Resistor_SMD:R_0402_1005Metric
- added L5: 5.6nH 0402, Inductor_SMD:L_0402_1005Metric, F.Cu at (31.7, 73.1)
- AE1: footprint RF_Antenna:Texas_SWRA117D_2.4GHz_Left -> RF_Antenna:Johanson_2450AT43F0100
- C14: value 0402 1pF -> 0402 0.8pF
- C15: value 100nF -> 100nF 0402
- C16: value 100pF -> 100pF 0402
- C17: value 1nF -> 820pF 0402 - DNP
- J5: value Conn_01x03_Male -> BM03B 3P; footprint Connector_PinHeader_2.54mm:PinHeader_1x03_P2.54mm_Vertical -> Connector_JST:JST_SUR_BM03B-SURS-TF_1x03-1MP_P0.80mm_Vertical
- Y1: value 32MHz 12pF -> 32MHz 12pF 2016-4P; footprint Crystal:Crystal_SMD_3225-4Pin_3.2x2.5mm -> Crystal:Crystal_SMD_2016-4Pin_2.0x1.6mm
- moved C10 77.3 mm to (32.0, 59.7), turned to 90 degrees
- moved J5 75.8 mm to (37.0, 66.6), turned to 180 degrees
- moved Y1 74.4 mm to (34.0, 59.3), turned to 180 degrees
- moved R6 74.3 mm to (35.1, 34.5)
- moved C2 74.1 mm to (34.3, 55.8)
- moved R5 74.1 mm to (38.1, 35.0)
- moved L4 74.0 mm to (42.6, 48.9)
- moved C17 73.9 mm to (32.0, 50.8)
- moved C22 73.9 mm to (40.4, 44.3)
- moved C3 73.9 mm to (40.4, 46.2)
- moved C7 73.9 mm to (33.6, 46.2)
- moved C9 73.9 mm to (31.9, 38.9)
- moved BT1 73.9 mm to (36.6, 40.6)
- moved C12 73.9 mm to (31.4, 31.8)
- moved C19 73.9 mm to (42.8, 33.0)
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Connections:
- C14 pad 2: VSS_PA -> GND
- C9 pad 1: 3.3VO -> +3V3
- J3 pad 1: GPIO15 -> unconnected-(J3-Pin_1-Pad1)
- J3 pad 10: GPIO8 -> unconnected-(J3-Pin_10-Pad10)
- J3 pad 11: GPIO7 -> unconnected-(J3-Pin_11-Pad11)
- J3 pad 12: GPIO6 -> unconnected-(J3-Pin_12-Pad12)
- J3 pad 13: GND -> unconnected-(J3-Pin_13-Pad13)
- J3 pad 14: GPIO5 -> unconnected-(J3-Pin_14-Pad14)
- J3 pad 15: GPIO4 -> unconnected-(J3-Pin_15-Pad15)
- J3 pad 16: GPIO3 -> unconnected-(J3-Pin_16-Pad16)
- J3 pad 17: GPIO2 -> unconnected-(J3-Pin_17-Pad17)
- J3 pad 18: GND -> unconnected-(J3-Pin_18-Pad18)
- J3 pad 19: GPIO1 -> unconnected-(J3-Pin_19-Pad19)
- J3 pad 2: GPIO14 -> unconnected-(J3-Pin_2-Pad2)
- J3 pad 20: GPIO0 -> unconnected-(J3-Pin_20-Pad20)
- J3 pad 3: GND -> unconnected-(J3-Pin_3-Pad3)
- J3 pad 4: GPIO13 -> unconnected-(J3-Pin_4-Pad4)
- J3 pad 5: GPIO12 -> unconnected-(J3-Pin_5-Pad5)
- J3 pad 6: GPIO11 -> unconnected-(J3-Pin_6-Pad6)
- J3 pad 7: GPIO10 -> unconnected-(J3-Pin_7-Pad7)
- J3 pad 8: GND -> unconnected-(J3-Pin_8-Pad8)
- J3 pad 9: GPIO9 -> unconnected-(J3-Pin_9-Pad9)
- J4 pad 1: VBUS -> unconnected-(J4-Pin_1-Pad1)
- J4 pad 10: GPIO23 -> unconnected-(J4-Pin_10-Pad10)
- J4 pad 11: RESET -> unconnected-(J4-Pin_11-Pad11)
- J4 pad 12: GPIO22 -> unconnected-(J4-Pin_12-Pad12)
- J4 pad 13: GND -> unconnected-(J4-Pin_13-Pad13)
- J4 pad 14: GPIO21 -> unconnected-(J4-Pin_14-Pad14)
- J4 pad 15: GPIO20 -> unconnected-(J4-Pin_15-Pad15)
- J4 pad 16: GPIO19 -> unconnected-(J4-Pin_16-Pad16)
- J4 pad 17: GPIO18 -> unconnected-(J4-Pin_17-Pad17)
- J4 pad 18: GND -> unconnected-(J4-Pin_18-Pad18)
- J4 pad 19: GPIO17 -> unconnected-(J4-Pin_19-Pad19)
- J4 pad 2: VSYS -> unconnected-(J4-Pin_2-Pad2)
- J4 pad 20: GPIO16 -> unconnected-(J4-Pin_20-Pad20)
- J4 pad 3: GND -> unconnected-(J4-Pin_3-Pad3)
- J4 pad 4: 3V3_EN -> unconnected-(J4-Pin_4-Pad4)
- J4 pad 5: 3.3VO -> unconnected-(J4-Pin_5-Pad5)
- J4 pad 6: GPIO26 -> unconnected-(J4-Pin_6-Pad6)
- J4 pad 7: GPIO25 -> unconnected-(J4-Pin_7-Pad7)
- J4 pad 8: GND -> unconnected-(J4-Pin_8-Pad8)
- J4 pad 9: GPIO24 -> unconnected-(J4-Pin_9-Pad9)
- L1 pad 2: 3.3VO -> +3V3
- U1 pad 4: 3.3VO -> +3V3
- U3 pad F23: VSS_PA -> GND
Routing:
- net GPIO0: track 27.4 -> 0.00 mm
- net GPIO15: track 25.3 -> 0.00 mm, vias 1 -> 0
- net GPIO1: track 24.8 -> 0.00 mm
- net GPIO16: track 24.3 -> 0.00 mm
- net GPIO14: track 22.6 -> 0.00 mm, vias 1 -> 0
- net 3.3VO: track 21.8 -> 0.00 mm, vias 1 -> 0
- net GPIO17: track 21.7 -> 0.00 mm
- net GPIO2: track 19.6 -> 0.00 mm
- net GPIO13: track 19.6 -> 0.00 mm, vias 1 -> 0
- net GPIO18: track 18.0 -> 0.00 mm
- net GPIO11: track 17.8 -> 0.00 mm, vias 1 -> 0
- net GPIO12: track 17.4 -> 0.00 mm, vias 3 -> 0
- net 3V3_EN: track 19.6 -> 3.00 mm, vias 1 -> 0
- net GPIO19: track 16.2 -> 0.00 mm
- net GPIO3: track 15.6 -> 0.00 mm
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Other:
- board size 21.2 x 57.7 mm -> 21.2 x 57.2 mm
- board text removed: "DEBUG"
- board text removed: "SWCLK"
- board text removed: "SWDIO"
- board text removed: "nRF52840 Prototype R#0.1"
